Commit message: feat: add ROS2 package and ESP32 hardware bridge
Convert the repo into an ament_python package, switch mesh paths to
package://, and add a hardware_bridge node that polls the ESP32 HTTP API
and publishes joint_states with finger mimic joints.
Co-authored-by: monkeycode-ai <monkeycode-ai@chaitin.com>

File: urdf/exoskeleton.urdf (robot description, URDF)
Before this commit: robot exoskeleton_hand, 22 links, 21 joints
Links:
- link base_link: geometry collision mesh filename=package://exoskeleton/meshes/BASE.STL scale=0.001 0.001 0.001; visual mesh filename=package://exoskeleton/meshes/BASE.STL scale=0.001 0.001 0.001
- link finger2_phalanx1: geometry collision mesh filename=package://exoskeleton/meshes/fingers/finger%202/a1.STL scale=0.001 0.001 0.001; visual mesh filename=package://exoskeleton/meshes/fingers/finger%202/a1.STL scale=0.001 0.001 0.001
- link finger2_phalanx2: geometry collision mesh filename=package://exoskeleton/meshes/fingers/finger%202/a2.STL scale=0.001 0.001 0.001; collision mesh filename=package://exoskeleton/meshes/fingers/finger%202/b1.STL scale=0.001 0.001 0.001
- link finger2_phalanx3: geometry collision mesh filename=package://exoskeleton/meshes/fingers/finger%202/a3.1.STL scale=0.001 0.001 0.001; collision mesh filename=package://exoskeleton/meshes/fingers/finger%202/a3.2.STL scale=0.001 0.001 0.001
- link finger2_phalanx4: geometry collision mesh filename=package://exoskeleton/meshes/fingers/finger%202/a4.STL scale=0.001 0.001 0.001; collision mesh filename=package://exoskeleton/meshes/fingers/finger%202/a5.1.STL scale=0.001 0.001 0.001
- link finger3_phalanx1: geometry collision mesh filename=package://exoskeleton/meshes/fingers/finger%203/a1.STL scale=0.001 0.001 0.001; visual mesh filename=package://exoskeleton/meshes/fingers/finger%203/a1.STL scale=0.001 0.001 0.001
- link finger3_phalanx2: geometry collision mesh filename=package://exoskeleton/meshes/fingers/finger%203/a2.STL scale=0.001 0.001 0.001; collision mesh filename=package://exoskeleton/meshes/fingers/finger%203/b1.STL scale=0.001 0.001 0.001
- link finger3_phalanx3: geometry collision mesh filename=package://exoskeleton/meshes/fingers/finger%203/a3.1.STL scale=0.001 0.001 0.001; collision mesh filename=package://exoskeleton/meshes/fingers/finger%203/a3.2.STL scale=0.001 0.001 0.001
- link finger3_phalanx4: geometry collision mesh filename=package://exoskeleton/meshes/fingers/finger%203/a4.STL scale=0.001 0.001 0.001; collision mesh filename=package://exoskeleton/meshes/fingers/finger%203/a5.1.STL scale=0.001 0.001 0.001
- link finger4_phalanx1: geometry collision mesh filename=package://exoskeleton/meshes/fingers/finger%204/a1.STL scale=0.001 0.001 0.001; visual mesh filename=package://exoskeleton/meshes/fingers/finger%204/a1.STL scale=0.001 0.001 0.001
- link finger4_phalanx2: geometry collision mesh filename=package://exoskeleton/meshes/fingers/finger%204/a2.STL scale=0.001 0.001 0.001; collision mesh filename=package://exoskeleton/meshes/fingers/finger%204/b1.STL scale=0.001 0.001 0.001
- link finger4_phalanx3: geometry collision mesh filename=package://exoskeleton/meshes/fingers/finger%204/a3.1.STL scale=0.001 0.001 0.001; collision mesh filename=package://exoskeleton/meshes/fingers/finger%204/a3.2.STL scale=0.001 0.001 0.001
- link finger4_phalanx4: geometry collision mesh filename=package://exoskeleton/meshes/fingers/finger%204/a4.STL scale=0.001 0.001 0.001; collision mesh filename=package://exoskeleton/meshes/fingers/finger%204/a5.1.STL scale=0.001 0.001 0.001
- link index_phalanx1: geometry collision mesh filename=package://exoskeleton/meshes/fingers/Index/INDEX%201.STL scale=0.001 0.001 0.001; visual mesh filename=package://exoskeleton/meshes/fingers/Index/INDEX%201.STL scale=0.001 0.001 0.001
- link index_phalanx2: geometry collision mesh filename=package://exoskeleton/meshes/fingers/Index/INDEX%202.STL scale=0.001 0.001 0.001; collision mesh filename=package://exoskeleton/meshes/fingers/Index/finger%201.1.STL scale=0.001 0.001 0.001
- link index_phalanx3: geometry collision mesh filename=package://exoskeleton/meshes/fingers/Index/INDEX%203.1.STL scale=0.001 0.001 0.001; collision mesh filename=package://exoskeleton/meshes/fingers/Index/INDEX%203.2.STL scale=0.001 0.001 0.001
- link index_phalanx4: geometry collision mesh filename=package://exoskeleton/meshes/fingers/Index/INDEX%204.STL scale=0.001 0.001 0.001; collision mesh filename=package://exoskeleton/meshes/fingers/Index/INDEX%205.1.STL scale=0.001 0.001 0.001
- link thumb_phalanx1: geometry collision mesh filename=package://exoskeleton/meshes/fingers/thumb/a1.STL scale=0.001 0.001 0.001; visual mesh filename=package://exoskeleton/meshes/fingers/thumb/a1.STL scale=0.001 0.001 0.001
- link thumb_phalanx2: geometry collision mesh filename=package://exoskeleton/meshes/fingers/thumb/a2.STL scale=0.001 0.001 0.001; collision mesh filename=package://exoskeleton/meshes/fingers/thumb/b1.STL scale=0.001 0.001 0.001
- link thumb_phalanx3: geometry collision mesh filename=package://exoskeleton/meshes/fingers/thumb/c1.1.STL scale=0.001 0.001 0.001; collision mesh filename=package://exoskeleton/meshes/fingers/thumb/c1.2.STL scale=0.001 0.001 0.001
- link thumb_phalanx4: geometry collision mesh filename=package://exoskeleton/meshes/fingers/thumb/a3.1.STL scale=0.001 0.001 0.001; collision mesh filename=package://exoskeleton/meshes/fingers/thumb/a3.2.STL scale=0.001 0.001 0.001
- link wrist_link: geometry collision mesh filename=package://exoskeleton/meshes/WRIST%20STARP.STL scale=0.001 0.001 0.001; visual mesh filename=package://exoskeleton/meshes/WRIST%20STARP.STL scale=0.001 0.001 0.001

File: urdf/exoskeleton_mj.urdf (robot description, URDF)
Before this commit: robot exoskeleton_hand, 22 links, 21 joints
Links:
- link base_link: geometry collision mesh filename=package://exoskeleton/meshes/BASE.STL scale=0.001 0.001 0.001; visual mesh filename=package://exoskeleton/meshes/BASE.STL scale=0.001 0.001 0.001
- link finger2_phalanx1: geometry collision mesh filename=package://exoskeleton/meshes/fingers/finger 2/a1.STL scale=0.001 0.001 0.001; visual mesh filename=package://exoskeleton/meshes/fingers/finger 2/a1.STL scale=0.001 0.001 0.001
- link finger2_phalanx2: geometry collision mesh filename=package://exoskeleton/meshes/fingers/finger 2/a2.STL scale=0.001 0.001 0.001; collision mesh filename=package://exoskeleton/meshes/fingers/finger 2/b1.STL scale=0.001 0.001 0.001
- link finger2_phalanx3: geometry collision mesh filename=package://exoskeleton/meshes/fingers/finger 2/a3.1.STL scale=0.001 0.001 0.001; collision mesh filename=package://exoskeleton/meshes/fingers/finger 2/a3.2.STL scale=0.001 0.001 0.001
- link finger2_phalanx4: geometry collision mesh filename=package://exoskeleton/meshes/fingers/finger 2/a4.STL scale=0.001 0.001 0.001; collision mesh filename=package://exoskeleton/meshes/fingers/finger 2/a5.1.STL scale=0.001 0.001 0.001
- link finger3_phalanx1: geometry collision mesh filename=package://exoskeleton/meshes/fingers/finger 3/a1.STL scale=0.001 0.001 0.001; visual mesh filename=package://exoskeleton/meshes/fingers/finger 3/a1.STL scale=0.001 0.001 0.001
- link finger3_phalanx2: geometry collision mesh filename=package://exoskeleton/meshes/fingers/finger 3/a2.STL scale=0.001 0.001 0.001; collision mesh filename=package://exoskeleton/meshes/fingers/finger 3/b1.STL scale=0.001 0.001 0.001
- link finger3_phalanx3: geometry collision mesh filename=package://exoskeleton/meshes/fingers/finger 3/a3.1.STL scale=0.001 0.001 0.001; collision mesh filename=package://exoskeleton/meshes/fingers/finger 3/a3.2.STL scale=0.001 0.001 0.001
- link finger3_phalanx4: geometry collision mesh filename=package://exoskeleton/meshes/fingers/finger 3/a4.STL scale=0.001 0.001 0.001; collision mesh filename=package://exoskeleton/meshes/fingers/finger 3/a5.1.STL scale=0.001 0.001 0.001
- link finger4_phalanx1: geometry collision mesh filename=package://exoskeleton/meshes/fingers/finger 4/a1.STL scale=0.001 0.001 0.001; visual mesh filename=package://exoskeleton/meshes/fingers/finger 4/a1.STL scale=0.001 0.001 0.001
- link finger4_phalanx2: geometry collision mesh filename=package://exoskeleton/meshes/fingers/finger 4/a2.STL scale=0.001 0.001 0.001; collision mesh filename=package://exoskeleton/meshes/fingers/finger 4/b1.STL scale=0.001 0.001 0.001
- link finger4_phalanx3: geometry collision mesh filename=package://exoskeleton/meshes/fingers/finger 4/a3.1.STL scale=0.001 0.001 0.001; collision mesh filename=package://exoskeleton/meshes/fingers/finger 4/a3.2.STL scale=0.001 0.001 0.001
- link finger4_phalanx4: geometry collision mesh filename=package://exoskeleton/meshes/fingers/finger 4/a4.STL scale=0.001 0.001 0.001; collision mesh filename=package://exoskeleton/meshes/fingers/finger 4/a5.1.STL scale=0.001 0.001 0.001
- link index_phalanx1: geometry collision mesh filename=package://exoskeleton/meshes/fingers/Index/INDEX 1.STL scale=0.001 0.001 0.001; visual mesh filename=package://exoskeleton/meshes/fingers/Index/INDEX 1.STL scale=0.001 0.001 0.001
- link index_phalanx2: geometry collision mesh filename=package://exoskeleton/meshes/fingers/Index/INDEX 2.STL scale=0.001 0.001 0.001; collision mesh filename=package://exoskeleton/meshes/fingers/Index/finger 1.1.STL scale=0.001 0.001 0.001
- link index_phalanx3: geometry collision mesh filename=package://exoskeleton/meshes/fingers/Index/INDEX 3.1.STL scale=0.001 0.001 0.001; collision mesh filename=package://exoskeleton/meshes/fingers/Index/INDEX 3.2.STL scale=0.001 0.001 0.001
- link index_phalanx4: geometry collision mesh filename=package://exoskeleton/meshes/fingers/Index/INDEX 4.STL scale=0.001 0.001 0.001; collision mesh filename=package://exoskeleton/meshes/fingers/Index/INDEX 5.1.STL scale=0.001 0.001 0.001
- link thumb_phalanx1: geometry collision mesh filename=package://exoskeleton/meshes/fingers/thumb/a1.STL scale=0.001 0.001 0.001; visual mesh filename=package://exoskeleton/meshes/fingers/thumb/a1.STL scale=0.001 0.001 0.001
- link thumb_phalanx2: geometry collision mesh filename=package://exoskeleton/meshes/fingers/thumb/a2.STL scale=0.001 0.001 0.001; collision mesh filename=package://exoskeleton/meshes/fingers/thumb/b1.STL scale=0.001 0.001 0.001
- link thumb_phalanx3: geometry collision mesh filename=package://exoskeleton/meshes/fingers/thumb/c1.1.STL scale=0.001 0.001 0.001; collision mesh filename=package://exoskeleton/meshes/fingers/thumb/c1.2.STL scale=0.001 0.001 0.001
- link thumb_phalanx4: geometry collision mesh filename=package://exoskeleton/meshes/fingers/thumb/a3.1.STL scale=0.001 0.001 0.001; collision mesh filename=package://exoskeleton/meshes/fingers/thumb/a3.2.STL scale=0.001 0.001 0.001
- link wrist_link: geometry collision mesh filename=package://exoskeleton/meshes/WRIST STARP.STL scale=0.001 0.001 0.001; visual mesh filename=package://exoskeleton/meshes/WRIST STARP.STL scale=0.001 0.001 0.001
